Commit message: Manual changes
Small manual changes to comply with URDF specifications.
Kept the problematic parts as comments.

File: urdf/AchileMKinect.urdf (robot description, URDF)
Before this commit: robot AchileMKinect, 40 links, 40 joints
Joints:
- removed joint HeadX
- removed joint Pelvis
- added joint rPoint: type prismatic, parent rRadius, child rRadius+rWristX, origin xyz=-0.007033 -0.430224 -0.446428 rpy=0 0 0, axis 1.000000 0.000000 0.000000, limit lower=-0.500000 upper=0.500000 effort=0 velocity=0
